File: Endonasal_Module_Breakout_rev1.sch (EAGLE design)
At the start: 43 parts, among them J1 CONN_RECT_2X12TH, J2 CONN_RECT_2X12TH, J3 CONN_RECT_2X32NOHOLES, J4 CONN_RECT_2X20TH, J5 JACK_8P8C_RJ45_ETHERNET, J6 CONN_RECT_2X10TH, J7 CONN_RECT_2X10TH, U1 OR_M3, U2 OR_M0

Commit message: Layout finished (hopefully)
Parts:
- C2, C7: value 0.1uF -> 10uF; device SparkFun-Capacitors:CAP0603-CAP -> Cannula_1_0:CAP0805
- C3, C8: value 10uF -> 0.1uF; device Cannula_1_0:CAP0805 -> SparkFun-Capacitors:CAP0603-CAP
- J1, J2: value CONN_RECT_2X12TH -> CONN_RECT_2X10TH; device Cannula_1_0:CONN_RECT_2X12TH -> Cannula_1_0:CONN_RECT_2X10TH
- J3: value CONN_RECT_2X32NOHOLES -> JACK_8P8C_RJ45_ETHERNET; device Cannula_1_0:CONN_RECT_2X32NOHOLES -> Cannula_1_0:JACK_8P8C_RJ45_ETHERNET
- J5: value JACK_8P8C_RJ45_ETHERNET -> CONN_RECT_2X32NOHOLES; device Cannula_1_0:JACK_8P8C_RJ45_ETHERNET -> Cannula_1_0:CONN_RECT_2X32NOHOLES
- J6, J7: value CONN_RECT_2X10TH -> CONN_RECT_2X12TH; device Cannula_1_0:CONN_RECT_2X10TH -> Cannula_1_0:CONN_RECT_2X12TH
- R1, R2, R3, R4, R5, R6: value 10K -> 1; device SparkFun-Passives:RESISTOR-ARRAY0603-ARV -> Cannula_1_0:RESISTOR-0603
- R10, R11, R12, R13, R14, R9: value 1 -> 10K; device Cannula_1_0:RESISTOR-0603 -> SparkFun-Passives:RESISTOR-ARRAY0603-ARV
- R7: value 220 -> 1
- R8: value 1 -> 220
- U1: value OR_M3 -> OR_M0
- U2: value OR_M0 -> OR_M3
- renumbered TP1 to 5V, TP2 to GND, TP3 to 5V-IN, TP4 to 3.3V, TP6 to 3.3V-IN
Connections:
- net 3.3V: now also C3.1, C8.1, C9.1, J6.14, J6.22, J6.6, J7.14, J7.22, J7.6, R7.1; no longer C1.1, C2.1, C7.1, J1.14, J1.22, J1.6, J2.14, J2.22, J2.6, R8.1
- net 3.3V_IN: now also J5.16, J5.26, J5.36, J5.46, J5.56, J5.6, R7.2; no longer J3.16, J3.26, J3.36, J3.46, J3.56, J3.6, R8.2
- net GND: now also J3.CASE, J5.10, J5.14, J5.20, J5.24, J5.30, J5.34, J5.4, J5.40, J5.44, J5.50, J5.54, J5.60, J6.12, J6.20, J6.4, J7.12, J7.20, J7.4; no longer J1.12, J1.20, J1.4, J2.12, J2.20, J2.4, J3.10, J3.14, J3.20, J3.24, J3.30, J3.34, J3.4, J3.40, J3.44, J3.50, J3.54, J3.60, J5.CASE
- net LIMIT1: now also J3.5, U1G$1.B; no longer J5.5, U2G$1.B
- net LIMIT2: now also J3.7, U1G$1.A, U2G$1.B; no longer J5.7, U1G$1.B, U2G$1.A
- net LIMIT3: now also J3.8, U2G$1.A; no longer J5.8, U1G$1.A
- net M0A: now also J1.5, J1.6; no longer J6.5, J6.6
- net M0B: now also J1.3, J1.4; no longer J6.3, J6.4
- net M0C: now also J1.1, J1.2; no longer J6.1, J6.2
- net M0_ENC_A: now also J5.7, J6.7; no longer J1.7, J3.7
- net M0_ENC_B: now also J5.8, J6.8; no longer J1.8, J3.8
- net M0_HALL1: now also J5.1, J6.1, R9C.2; no longer J1.1, J3.1, R1C.2
- net M0_HALL2: now also J5.2, J6.2, R9B.2; no longer J1.2, J3.2, R1B.2
- net M0_HALL3: now also J5.3, J6.3, R9A.2; no longer J1.3, J3.3, R1A.2
- net M0_LIMIT: now also J5.9, U1G$1.Y; no longer J3.9, U2G$1.Y
- net M0_VHALL: now also C1.1, J3.1, J6.5, R1.1, R8.2, R9A.1, R9B.1, R9C.1; no longer C9.1, J1.5, J5.1, R14.1, R1A.1, R1B.1, R1C.1, R7.2
- net M0_VHALL_IN: now also J5.5, R1.2; no longer J3.5, R14.2
- net M1A: now also J1.12, J1.13; no longer J6.12, J6.13
- net M1B: now also J1.10, J1.11; no longer J6.10, J6.11
- net M1C: now also J1.8, J1.9; no longer J6.8, J6.9
- net M1_ENC_A: now also J5.17, J6.15; no longer J1.15, J3.17
- net M1_ENC_B: now also J5.18, J6.16; no longer J1.16, J3.18
- net M1_HALL1: now also J5.11, J6.9, R10C.1; no longer J1.9, J3.11, R2C.1
- net M1_HALL2: now also J5.12, J6.10, R10B.1; no longer J1.10, J3.12, R2B.1
- net M1_HALL3: now also J5.13, J6.11, R10A.1; no longer J1.11, J3.13, R2A.1
- net M1_LIMIT: now also J5.19; no longer J3.19
- net M1_VHALL: now also C2.1, J6.13, R10A.2, R10B.2, R10C.2, R2.1; no longer C8.1, J1.13, R13.1, R2A.2, R2B.2, R2C.2
- net M1_VHALL_IN: now also J5.15, R2.2; no longer J3.15, R13.2
- net M2A: now also J1.19, J1.20; no longer J6.19, J6.20
- net M2B: now also J1.17, J1.18; no longer J6.17, J6.18
- net M2C: now also J1.15, J1.16; no longer J6.15, J6.16
- net M2_ENC_A: now also J5.27, J6.23; no longer J1.23, J3.27
- net M2_ENC_B: now also J5.28, J6.24; no longer J1.24, J3.28
- net M2_HALL1: now also J5.21, J6.17, R11B.1; no longer J1.17, J3.21, R3B.1
- net M2_HALL2: now also J5.22, J6.18, R11C.1; no longer J1.18, J3.22, R3C.1
- net M2_HALL3: now also J5.23, J6.19, R11A.1; no longer J1.19, J3.23, R3A.1
- net M2_LIMIT: now also J5.29; no longer J3.29
- net M2_VHALL: now also C4.1, J6.21, R11A.2, R11B.2, R11C.2, R3.1; no longer C6.1, J1.21, R12.1, R3A.2, R3B.2, R3C.2
- net M2_VHALL_IN: now also J5.25, R3.2; no longer J3.25, R12.2
- net M3A: now also J2.5, J2.6; no longer J7.5, J7.6
- net M3B: now also J2.3, J2.4; no longer J7.3, J7.4
- net M3C: now also J2.1, J2.2; no longer J7.1, J7.2
- net M3_ENC_A: now also J5.37, J7.7; no longer J2.7, J3.37
- net M3_ENC_B: now also J5.38, J7.8; no longer J2.8, J3.38
- net M3_HALL1: now also J5.31, J7.1, R12A.1; no longer J2.1, J3.31, R4A.1
- net M3_HALL2: now also J5.32, J7.2, R12B.1; no longer J2.2, J3.32, R4B.1
- net M3_HALL3: now also J5.33, J7.3, R12C.1; no longer J2.3, J3.33, R4C.1
- net M3_LIMIT: now also J5.39, U2G$1.Y; no longer J3.39, U1G$1.Y
- net M3_VHALL: now also J7.5, R12A.2, R12B.2, R12C.2, R4.1; no longer J2.5, R11.1, R4A.2, R4B.2, R4C.2
- net M3_VHALL_IN: now also J5.35, R4.2; no longer J3.35, R11.2
- net M4A: now also J2.12, J2.13; no longer J7.12, J7.13
- net M4B: now also J2.10, J2.11; no longer J7.10, J7.11
- net M4C: now also J2.8, J2.9; no longer J7.8, J7.9
- net M4_ENC_A: now also J5.47, J7.15; no longer J2.15, J3.47
- net M4_ENC_B: now also J5.48, J7.16; no longer J2.16, J3.48
- net M4_HALL1: now also J5.41, J7.9, R13A.1; no longer J2.9, J3.41, R5A.1
- net M4_HALL2: now also J5.42, J7.10, R13B.1; no longer J2.10, J3.42, R5B.1
- net M4_HALL3: now also J5.43, J7.11, R13C.1; no longer J2.11, J3.43, R5C.1
- net M4_LIMIT: now also J5.49; no longer J3.49
- net M4_VHALL: now also C6.1, J7.13, R13A.2, R13B.2, R13C.2, R5.1; no longer C4.1, J2.13, R10.1, R5A.2, R5B.2, R5C.2
- net M4_VHALL_IN: now also J5.45, R5.2; no longer J3.45, R10.2
- net M5A: now also J2.19, J2.20; no longer J7.19, J7.20
- net M5B: now also J2.17, J2.18; no longer J7.17, J7.18
- net M5C: now also J2.15, J2.16; no longer J7.15, J7.16
- net M5_ENC_A: now also J5.57, J7.23; no longer J2.23, J3.57
- net M5_ENC_B: now also J5.58, J7.24; no longer J2.24, J3.58
- net M5_HALL1: now also J5.51, J7.17, R14B.1; no longer J2.17, J3.51, R6B.1
- net M5_HALL2: now also J5.52, J7.18, R14A.1; no longer J2.18, J3.52, R6A.1
- net M5_HALL3: now also J5.53, J7.19, R14C.1; no longer J2.19, J3.53, R6C.1
- net M5_LIMIT: now also J5.59; no longer J3.59
- net M5_VHALL: now also C7.1, J7.21, R14A.2, R14B.2, R14C.2, R6.1; no longer C3.1, J2.21, R6A.2, R6B.2, R6C.2, R9.1
- net M5_VHALL_IN: now also J5.55, R6.2; no longer J3.55, R9.2
- net N$190: now also J5.62; no longer J3.62
- net N$191: now also J5.63; no longer J3.63
- net N$192: now also J5.64; no longer J3.64
- net N$6: now also R8.1; no longer R7.1
Other:
- moved on the sheet: C1, C2, C3, C4, C6, C7, C8, C9, R7, R8, U1G$1, U1G$2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
